Commit message: update

File: urdf/susan_description.xacro (robot description, xacro)
@@ -1,3 +1,3 @@
-<robot name="onshape">
+<robot name="susan">
 <link name="link1">
 <visual>
@@ -519,5 +519,5 @@
 <link name="link2_right">
 <visual>
-<origin xyz="2.4651903288156618919e-32 -0.021000000000000004774 -0.04700000000000000705" rpy="1.570796326794896558 1.0024047512732148535e-32 -1.2325951644078253408e-30" />
+<origin xyz="0 -0.021000000000000001305 -0.04700000000000000705" rpy="1.570796326794896558 4.3908883778532081263e-33 1.1749307662810900005e-46" />
 <geometry>
 <mesh filename="package://susan_description/meshes/bracket_type_a.stl"/>
@@ -528,5 +528,5 @@
 </visual>
 <collision>
-<origin xyz="2.4651903288156618919e-32 -0.021000000000000004774 -0.04700000000000000705" rpy="1.570796326794896558 1.0024047512732148535e-32 -1.2325951644078253408e-30" />
+<origin xyz="0 -0.021000000000000001305 -0.04700000000000000705" rpy="1.570796326794896558 4.3908883778532081263e-33 1.1749307662810900005e-46" />
 <geometry>
 <mesh filename="package://susan_description/meshes/bracket_type_a.stl"/>
@@ -534,5 +534,5 @@
 </collision>
 <visual>
-<origin xyz="1.3267518160498689285e-15 -0.0022999999999988637173 -0.047000000000000048683" rpy="1.570796326794896558 2.2208773040168372319e-16 1.5707963267948341635" />
+<origin xyz="1.3263601752762148032e-15 -0.0022999999999988697888 -0.047000000000000034805" rpy="1.570796326794896558 2.2208773040168411762e-16 1.5707963267948341635" />
 <geometry>
 <mesh filename="package://susan_description/meshes/mg6012-i36v3-31.stl"/>
@@ -543,5 +543,5 @@
 </visual>
 <collision>
-<origin xyz="1.3267518160498689285e-15 -0.0022999999999988637173 -0.047000000000000048683" rpy="1.570796326794896558 2.2208773040168372319e-16 1.5707963267948341635" />
+<origin xyz="1.3263601752762148032e-15 -0.0022999999999988697888 -0.047000000000000034805" rpy="1.570796326794896558 2.2208773040168411762e-16 1.5707963267948341635" />
 <geometry>
 <mesh filename="package://susan_description/meshes/mg6012-i36v3-31.stl"/>
@@ -549,5 +549,5 @@
 </collision>
 <visual>
-<origin xyz="1.3267518160498689285e-15 -0.0022999999999988637173 -0.047000000000000048683" rpy="1.570796326794896558 2.2208773040168372319e-16 1.5707963267948341635" />
+<origin xyz="1.3263601752762148032e-15 -0.0022999999999988697888 -0.047000000000000034805" rpy="1.570796326794896558 2.2208773040168411762e-16 1.5707963267948341635" />
 <geometry>
 <mesh filename="package://susan_description/meshes/mg6012-i36v3-18.stl"/>
@@ -558,5 +558,5 @@
 </visual>
 <collision>
-<origin xyz="1.3267518160498689285e-15 -0.0022999999999988637173 -0.047000000000000048683" rpy="1.570796326794896558 2.2208773040168372319e-16 1.5707963267948341635" />
+<origin xyz="1.3263601752762148032e-15 -0.0022999999999988697888 -0.047000000000000034805" rpy="1.570796326794896558 2.2208773040168411762e-16 1.5707963267948341635" />
 <geometry>
 <mesh filename="package://susan_description/meshes/mg6012-i36v3-18.stl"/>
@@ -564,5 +564,5 @@
 </collision>
 <visual>
-<origin xyz="1.3267518160498689285e-15 -0.0022999999999988637173 -0.047000000000000048683" rpy="1.570796326794896558 2.2208773040168372319e-16 1.5707963267948341635" />
+<origin xyz="1.3263601752762148032e-15 -0.0022999999999988697888 -0.047000000000000034805" rpy="1.570796326794896558 2.2208773040168411762e-16 1.5707963267948341635" />
 <geometry>
 <mesh filename="package://susan_description/meshes/mg6012-i36v3-27.stl"/>
@@ -573,5 +573,5 @@
 </visual>
 <collision>
-<origin xyz="1.3267518160498689285e-15 -0.0022999999999988637173 -0.047000000000000048683" rpy="1.570796326794896558 2.2208773040168372319e-16 1.5707963267948341635" />
+<origin xyz="1.3263601752762148032e-15 -0.0022999999999988697888 -0.047000000000000034805" rpy="1.570796326794896558 2.2208773040168411762e-16 1.5707963267948341635" />
 <geometry>
 <mesh filename="package://susan_description/meshes/mg6012-i36v3-27.stl"/>
@@ -579,5 +579,5 @@
 </collision>
 <visual>
-<origin xyz="1.3267518160498689285e-15 -0.0022999999999988637173 -0.047000000000000048683" rpy="1.570796326794896558 2.2208773040168372319e-16 1.5707963267948341635" />
+<origin xyz="1.3263601752762148032e-15 -0.0022999999999988697888 -0.047000000000000034805" rpy="1.570796326794896558 2.2208773040168411762e-16 1.5707963267948341635" />
 <geometry>
 <mesh filename="package://susan_description/meshes/mg6012-i36v3-2.stl"/>
@@ -588,5 +588,5 @@
 </visual>
 <collision>
-<origin xyz="1.3267518160498689285e-15 -0.0022999999999988637173 -0.047000000000000048683" rpy="1.570796326794896558 2.2208773040168372319e-16 1.5707963267948341635" />
+<origin xyz="1.3263601752762148032e-15 -0.0022999999999988697888 -0.047000000000000034805" rpy="1.570796326794896558 2.2208773040168411762e-16 1.5707963267948341635" />
 <geometry>
 <mesh filename="package://susan_description/meshes/mg6012-i36v3-2.stl"/>
@@ -594,5 +594,5 @@
 </collision>
 <visual>
-<origin xyz="1.3267518160498689285e-15 -0.0022999999999988637173 -0.047000000000000048683" rpy="1.570796326794896558 2.2208773040168372319e-16 1.5707963267948341635" />
+<origin xyz="1.3263601752762148032e-15 -0.0022999999999988697888 -0.047000000000000034805" rpy="1.570796326794896558 2.2208773040168411762e-16 1.5707963267948341635" />
 <geometry>
 <mesh filename="package://susan_description/meshes/mg6012-i36v3-22.stl"/>
@@ -603,5 +603,5 @@
 </visual>
 <collision>
-<origin xyz="1.3267518160498689285e-15 -0.0022999999999988637173 -0.047000000000000048683" rpy="1.570796326794896558 2.2208773040168372319e-16 1.5707963267948341635" />
+<origin xyz="1.3263601752762148032e-15 -0.0022999999999988697888 -0.047000000000000034805" rpy="1.570796326794896558 2.2208773040168411762e-16 1.5707963267948341635" />
 <geometry>
 <mesh filename="package://susan_description/meshes/mg6012-i36v3-22.stl"/>
@@ -609,5 +609,5 @@
 </collision>
 <visual>
-<origin xyz="1.3267518160498689285e-15 -0.0022999999999988637173 -0.047000000000000048683" rpy="1.570796326794896558 2.2208773040168372319e-16 1.5707963267948341635" />
+<origin xyz="1.3263601752762148032e-15 -0.0022999999999988697888 -0.047000000000000034805" rpy="1.570796326794896558 2.2208773040168411762e-16 1.5707963267948341635" />
 <geometry>
 <mesh filename="package://susan_description/meshes/mg6012-i36v3-21.stl"/>
@@ -618,5 +618,5 @@
 </visual>
 <collision>
-<origin xyz="1.3267518160498689285e-15 -0.0022999999999988637173 -0.047000000000000048683" rpy="1.570796326794896558 2.2208773040168372319e-16 1.5707963267948341635" />
+<origin xyz="1.3263601752762148032e-15 -0.0022999999999988697888 -0.047000000000000034805" rpy="1.570796326794896558 2.2208773040168411762e-16 1.5707963267948341635" />
 <geometry>
 <mesh filename="package://susan_description/meshes/mg6012-i36v3-21.stl"/>
@@ -624,5 +624,5 @@
 </collision>
 <visual>
-<origin xyz="1.3267518160498689285e-15 -0.0022999999999988637173 -0.047000000000000048683" rpy="1.570796326794896558 2.2208773040168372319e-16 1.5707963267948341635" />
+<origin xyz="1.3263601752762148032e-15 -0.0022999999999988697888 -0.047000000000000034805" rpy="1.570796326794896558 2.2208773040168411762e-16 1.5707963267948341635" />
 <geometry>
 <mesh filename="package://susan_description/meshes/mg6012-i36v3-7.stl"/>
@@ -633,5 +633,5 @@
 </visual>
 <collision>
-<origin xyz="1.3267518160498689285e-15 -0.0022999999999988637173 -0.047000000000000048683" rpy="1.570796326794896558 2.2208773040168372319e-16 1.5707963267948341635" />
+<origin xyz="1.3263601752762148032e-15 -0.0022999999999988697888 -0.047000000000000034805" rpy="1.570796326794896558 2.2208773040168411762e-16 1.5707963267948341635" />
 <geometry>
 <mesh filename="package://susan_description/meshes/mg6012-i36v3-7.stl"/>
@@ -639,5 +639,5 @@
 </collision>
 <visual>
-<origin xyz="1.3267518160498689285e-15 -0.0022999999999988637173 -0.047000000000000048683" rpy="1.570796326794896558 2.2208773040168372319e-16 1.5707963267948341635" />
+<origin xyz="1.3263601752762148032e-15 -0.0022999999999988697888 -0.047000000000000034805" rpy="1.570796326794896558 2.2208773040168411762e-16 1.5707963267948341635" />
 <geometry>
 <mesh filename="package://susan_description/meshes/mg6012-i36v3-6.stl"/>
@@ -648,5 +648,5 @@
 </visual>
 <collision>
-<origin xyz="1.3267518160498689285e-15 -0.0022999999999988637173 -0.047000000000000048683" rpy="1.570796326794896558 2.2208773040168372319e-16 1.5707963267948341635" />
+<origin xyz="1.3263601752762148032e-15 -0.0022999999999988697888 -0.047000000000000034805" rpy="1.570796326794896558 2.2208773040168411762e-16 1.5707963267948341635" />
 <geometry>
 <mesh filename="package://susan_description/meshes/mg6012-i36v3-6.stl"/>
@@ -654,5 +654,5 @@
 </collision>
 <visual>
-<origin xyz="1.3267518160498689285e-15 -0.0022999999999988637173 -0.047000000000000048683" rpy="1.570796326794896558 2.2208773040168372319e-16 1.5707963267948341635" />
+<origin xyz="1.3263601752762148032e-15 -0.0022999999999988697888 -0.047000000000000034805" rpy="1.570796326794896558 2.2208773040168411762e-16 1.5707963267948341635" />
 <geometry>
 <mesh filename="package://susan_description/meshes/mg6012-i36v3-11.stl"/>
@@ -663,5 +663,5 @@
 </visual>
 <collision>
-<origin xyz="1.3267518160498689285e-15 -0.0022999999999988637173 -0.047000000000000048683" rpy="1.570796326794896558 2.2208773040168372319e-16 1.5707963267948341635" />
+<origin xyz="1.3263601752762148032e-15 -0.0022999999999988697888 -0.047000000000000034805" rpy="1.570796326794896558 2.2208773040168411762e-16 1.5707963267948341635" />
 <geometry>
 <mesh filename="package://susan_description/meshes/mg6012-i36v3-11.stl"/>
@@ -669,5 +669,5 @@
 </collision>
 <visual>
-<origin xyz="1.3267518160498689285e-15 -0.0022999999999988637173 -0.047000000000000048683" rpy="1.570796326794896558 2.2208773040168372319e-16 1.5707963267948341635" />
+<origin xyz="1.3263601752762148032e-15 -0.0022999999999988697888 -0.047000000000000034805" rpy="1.570796326794896558 2.2208773040168411762e-16 1.5707963267948341635" />
 <geometry>
 <mesh filename="package://susan_description/meshes/mg6012-i36v3-10.stl"/>
@@ -678,5 +678,5 @@
 </visual>
 <collision>
-<origin xyz="1.3267518160498689285e-15 -0.0022999999999988637173 -0.047000000000000048683" rpy="1.570796326794896558 2.2208773040168372319e-16 1.5707963267948341635" />
+<origin xyz="1.3263601752762148032e-15 -0.0022999999999988697888 -0.047000000000000034805" rpy="1.570796326794896558 2.2208773040168411762e-16 1.5707963267948341635" />
 <geometry>
 <mesh filename="package://susan_description/meshes/mg6012-i36v3-10.stl"/>
@@ -684,5 +684,5 @@
 </collision>
 <visual>
-<origin xyz="1.3267518160498689285e-15 -0.0022999999999988637173 -0.047000000000000048683" rpy="1.570796326794896558 2.2208773040168372319e-16 1.5707963267948341635" />
+<origin xyz="1.3263601752762148032e-15 -0.0022999999999988697888 -0.047000000000000034805" rpy="1.570796326794896558 2.2208773040168411762e-16 1.5707963267948341635" />
 <geometry>
 <mesh filename="package://susan_description/meshes/mg6012-i36v3-16.stl"/>
@@ -693,5 +693,5 @@
 </visual>
 <collision>
-<origin xyz="1.3267518160498689285e-15 -0.0022999999999988637173 -0.047000000000000048683" rpy="1.570796326794896558 2.2208773040168372319e-16 1.5707963267948341635" />
+<origin xyz="1.3263601752762148032e-15 -0.0022999999999988697888 -0.047000000000000034805" rpy="1.570796326794896558 2.2208773040168411762e-16 1.5707963267948341635" />
 <geometry>
 <mesh filename="package://susan_description/meshes/mg6012-i36v3-16.stl"/>
@@ -699,5 +699,5 @@
 </collision>
 <visual>
-<origin xyz="1.3267518160498689285e-15 -0.0022999999999988637173 -0.047000000000000048683" rpy="1.570796326794896558 2.2208773040168372319e-16 1.5707963267948341635" />
+<origin xyz="1.3263601752762148032e-15 -0.0022999999999988697888 -0.047000000000000034805" rpy="1.570796326794896558 2.2208773040168411762e-16 1.5707963267948341635" />
 <geometry>
 <mesh filename="package://susan_description/meshes/mg6012-i36v3-29.stl"/>
@@ -708,5 +708,5 @@
 </visual>
 <collision>
-<origin xyz="1.3267518160498689285e-15 -0.0022999999999988637173 -0.047000000000000048683" rpy="1.570796326794896558 2.2208773040168372319e-16 1.5707963267948341635" />
+<origin xyz="1.3263601752762148032e-15 -0.0022999999999988697888 -0.047000000000000034805" rpy="1.570796326794896558 2.2208773040168411762e-16 1.5707963267948341635" />
 <geometry>
 <mesh filename="package://susan_description/meshes/mg6012-i36v3-29.stl"/>
@@ -714,5 +714,5 @@
 </collision>
 <visual>
-<origin xyz="1.3267518160498689285e-15 -0.0022999999999988637173 -0.047000000000000048683" rpy="1.570796326794896558 2.2208773040168372319e-16 1.5707963267948341635" />
+<origin xyz="1.3263601752762148032e-15 -0.0022999999999988697888 -0.047000000000000034805" rpy="1.570796326794896558 2.2208773040168411762e-16 1.5707963267948341635" />
 <geometry>
 <mesh filename="package://susan_description/meshes/mg6012-i36v3-17.stl"/>
@@ -723,5 +723,5 @@
 </visual>
 <collision>
-<origin xyz="1.3267518160498689285e-15 -0.0022999999999988637173 -0.047000000000000048683" rpy="1.570796326794896558 2.2208773040168372319e-16 1.5707963267948341635" />
+<origin xyz="1.3263601752762148032e-15 -0.0022999999999988697888 -0.047000000000000034805" rpy="1.570796326794896558 2.2208773040168411762e-16 1.5707963267948341635" />
 <geometry>
 <mesh filename="package://susan_description/meshes/mg6012-i36v3-17.stl"/>
@@ -729,5 +729,5 @@
 </collision>
 <visual>
-<origin xyz="1.3267518160498689285e-15 -0.0022999999999988637173 -0.047000000000000048683" rpy="1.570796326794896558 2.2208773040168372319e-16 1.5707963267948341635" />
+<origin xyz="1.3263601752762148032e-15 -0.0022999999999988697888 -0.047000000000000034805" rpy="1.570796326794896558 2.2208773040168411762e-16 1.5707963267948341635" />
 <geometry>
 <mesh filename="package://susan_description/meshes/mg6012-i36v3-34.stl"/>
@@ -738,5 +738,5 @@
 </visual>
 <collision>
-<origin xyz="1.3267518160498689285e-15 -0.0022999999999988637173 -0.047000000000000048683" rpy="1.570796326794896558 2.2208773040168372319e-16 1.5707963267948341635" />
+<origin xyz="1.3263601752762148032e-15 -0.0022999999999988697888 -0.047000000000000034805" rpy="1.570796326794896558 2.2208773040168411762e-16 1.5707963267948341635" />
 <geometry>
 <mesh filename="package://susan_description/meshes/mg6012-i36v3-34.stl"/>
@@ -744,5 +744,5 @@
 </collision>
 <visual>
-<origin xyz="1.3267518160498689285e-15 -0.0022999999999988637173 -0.047000000000000048683" rpy="1.570796326794896558 2.2208773040168372319e-16 1.5707963267948341635" />
+<origin xyz="1.3263601752762148032e-15 -0.0022999999999988697888 -0.047000000000000034805" rpy="1.570796326794896558 2.2208773040168411762e-16 1.5707963267948341635" />
 <geometry>
 <mesh filename="package://susan_description/meshes/mg6012-i36v3-28.stl"/>
@@ -753,5 +753,5 @@
 </visual>
 <collision>
-<origin xyz="1.3267518160498689285e-15 -0.0022999999999988637173 -0.047000000000000048683" rpy="1.570796326794896558 2.2208773040168372319e-16 1.5707963267948341635" />
+<origin xyz="1.3263601752762148032e-15 -0.0022999999999988697888 -0.047000000000000034805" rpy="1.570796326794896558 2.2208773040168411762e-16 1.5707963267948341635" />
 <geometry>
 <mesh filename="package://susan_description/meshes/mg6012-i36v3-28.stl"/>
@@ -759,5 +759,5 @@
 </collision>
 <visual>
-<origin xyz="1.3267518160498689285e-15 -0.0022999999999988637173 -0.047000000000000048683" rpy="1.570796326794896558 2.2208773040168372319e-16 1.5707963267948341635" />
+<origin xyz="1.3263601752762148032e-15 -0.0022999999999988697888 -0.047000000000000034805" rpy="1.570796326794896558 2.2208773040168411762e-16 1.5707963267948341635" />
 <geometry>
 <mesh filename="package://susan_description/meshes/mg6012-i36v3-25.stl"/>
@@ -768,5 +768,5 @@
 </visual>
 <collision>
-<origin xyz="1.3267518160498689285e-15 -0.0022999999999988637173 -0.047000000000000048683" rpy="1.570796326794896558 2.2208773040168372319e-16 1.5707963267948341635" />
+<origin xyz="1.3263601752762148032e-15 -0.0022999999999988697888 -0.047000000000000034805" rpy="1.570796326794896558 2.2208773040168411762e-16 1.5707963267948341635" />
 <geometry>
 <mesh filename="package://susan_description/meshes/mg6012-i36v3-25.stl"/>
@@ -774,5 +774,5 @@
 </collision>
 <visual>
-<origin xyz="1.3267518160498689285e-15 -0.0022999999999988637173 -0.047000000000000048683" rpy="1.570796326794896558 2.2208773040168372319e-16 1.5707963267948341635" />
+<origin xyz="1.3263601752762148032e-15 -0.0022999999999988697888 -0.047000000000000034805" rpy="1.570796326794896558 2.2208773040168411762e-16 1.5707963267948341635" />
 <geometry>
 <mesh filename="package://susan_description/meshes/mg6012-i36v3-19.stl"/>
@@ -783,5 +783,5 @@
 </visual>
 <collision>
-<origin xyz="1.3267518160498689285e-15 -0.0022999999999988637173 -0.047000000000000048683" rpy="1.570796326794896558 2.2208773040168372319e-16 1.5707963267948341635" />
+<origin xyz="1.3263601752762148032e-15 -0.0022999999999988697888 -0.047000000000000034805" rpy="1.570796326794896558 2.2208773040168411762e-16 1.5707963267948341635" />
 <geometry>
 <mesh filename="package://susan_description/meshes/mg6012-i36v3-19.stl"/>
@@ -789,5 +789,5 @@
 </collision>
 <visual>
-<origin xyz="1.3267518160498689285e-15 -0.0022999999999988637173 -0.047000000000000048683" rpy="1.570796326794896558 2.2208773040168372319e-16 1.5707963267948341635" />
+<origin xyz="1.3263601752762148032e-15 -0.0022999999999988697888 -0.047000000000000034805" rpy="1.570796326794896558 2.2208773040168411762e-16 1.5707963267948341635" />
 <geometry>
 <mesh filename="package://susan_description/meshes/mg6012-i36v3-24.stl"/>
@@ -798,5 +798,5 @@
 </visual>
 <collision>
-<origin xyz="1.3267518160498689285e-15 -0.0022999999999988637173 -0.047000000000000048683" rpy="1.570796326794896558 2.2208773040168372319e-16 1.5707963267948341635" />
+<origin xyz="1.3263601752762148032e-15 -0.0022999999999988697888 -0.047000000000000034805" rpy="1.570796326794896558 2.2208773040168411762e-16 1.5707963267948341635" />
 <geometry>
 <mesh filename="package://susan_description/meshes/mg6012-i36v3-24.stl"/>
@@ -804,5 +804,5 @@
 </collision>
 <visual>
-<origin xyz="1.3267518160498689285e-15 -0.0022999999999988637173 -0.047000000000000048683" rpy="1.570796326794896558 2.2208773040168372319e-16 1.5707963267948341635" />
+<origin xyz="1.3263601752762148032e-15 -0.0022999999999988697888 -0.047000000000000034805" rpy="1.570796326794896558 2.2208773040168411762e-16 1.5707963267948341635" />
 <geometry>
 <mesh filename="package://susan_description/meshes/mg6012-i36v3-4.stl"/>
@@ -813,5 +813,5 @@
 </visual>
 <collision>
-<origin xyz="1.3267518160498689285e-15 -0.0022999999999988637173 -0.047000000000000048683" rpy="1.570796326794896558 2.2208773040168372319e-16 1.5707963267948341635" />
+<origin xyz="1.3263601752762148032e-15 -0.0022999999999988697888 -0.047000000000000034805" rpy="1.570796326794896558 2.2208773040168411762e-16 1.5707963267948341635" />
 <geometry>
 <mesh filename="package://susan_description/meshes/mg6012-i36v3-4.stl"/>
@@ -819,5 +819,5 @@
 </collision>
 <visual>
-<origin xyz="1.3267518160498689285e-15 -0.0022999999999988637173 -0.047000000000000048683" rpy="1.570796326794896558 2.2208773040168372319e-16 1.5707963267948341635" />
+<origin xyz="1.3263601752762148032e-15 -0.0022999999999988697888 -0.047000000000000034805" rpy="1.570796326794896558 2.2208773040168411762e-16 1.5707963267948341635" />
 <geometry>
 <mesh filename="package://susan_description/meshes/mg6012-i36v3-8.stl"/>
@@ -828,5 +828,5 @@
 </visual>
 <collision>
-<origin xyz="1.3267518160498689285e-15 -0.0022999999999988637173 -0.047000000000000048683" rpy="1.570796326794896558 2.2208773040168372319e-16 1.5707963267948341635" />
+<origin xyz="1.3263601752762148032e-15 -0.0022999999999988697888 -0.047000000000000034805" rpy="1.570796326794896558 2.2208773040168411762e-16 1.5707963267948341635" />
 <geometry>
 <mesh filename="package://susan_description/meshes/mg6012-i36v3-8.stl"/>
@@ -834,5 +834,5 @@
 </collision>
 <visual>
-<origin xyz="1.3267518160498689285e-15 -0.0022999999999988637173 -0.047000000000000048683" rpy="1.570796326794896558 2.2208773040168372319e-16 1.5707963267948341635" />
+<origin xyz="1.3263601752762148032e-15 -0.0022999999999988697888 -0.047000000000000034805" rpy="1.570796326794896558 2.2208773040168411762e-16 1.5707963267948341635" />
 <geometry>
 <mesh filename="package://susan_description/meshes/mg6012-i36v3-20.stl"/>
@@ -843,5 +843,5 @@
 </visual>
 <collision>
-<origin xyz="1.3267518160498689285e-15 -0.0022999999999988637173 -0.047000000000000048683" rpy="1.570796326794896558 2.2208773040168372319e-16 1.5707963267948341635" />
+<origin xyz="1.3263601752762148032e-15 -0.0022999999999988697888 -0.047000000000000034805" rpy="1.570796326794896558 2.2208773040168411762e-16 1.5707963267948341635" />
 <geometry>
 <mesh filename="package://susan_description/meshes/mg6012-i36v3-20.stl"/>
@@ -849,5 +849,5 @@
 </collision>
 <visual>
-<origin xyz="1.3267518160498689285e-15 -0.0022999999999988637173 -0.047000000000000048683" rpy="1.570796326794896558 2.2208773040168372319e-16 1.5707963267948341635" />
+<origin xyz="1.3263601752762148032e-15 -0.0022999999999988697888 -0.047000000000000034805" rpy="1.570796326794896558 2.2208773040168411762e-16 1.5707963267948341635" />
 <geometry>
 <mesh filename="package://susan_description/meshes/mg6012-i36v3-12.stl"/>
@@ -858,5 +858,5 @@
 </visual>
 <collision>
-<origin xyz="1.3267518160498689285e-15 -0.0022999999999988637173 -0.047000000000000048683" rpy="1.570796326794896558 2.2208773040168372319e-16 1.5707963267948341635" />
+<origin xyz="1.3263601752762148032e-15 -0.0022999999999988697888 -0.047000000000000034805" rpy="1.570796326794896558 2.2208773040168411762e-16 1.5707963267948341635" />
 <geometry>
 <mesh filename="package://susan_description/meshes/mg6012-i36v3-12.stl"/>
@@ -864,5 +864,5 @@
 </collision>
 <visual>
-<origin xyz="1.3267518160498689285e-15 -0.0022999999999988637173 -0.047000000000000048683" rpy="1.570796326794896558 2.2208773040168372319e-16 1.5707963267948341635" />
+<origin xyz="1.3263601752762148032e-15 -0.0022999999999988697888 -0.047000000000000034805" rpy="1.570796326794896558 2.2208773040168411762e-16 1.5707963267948341635" />
 <geometry>
 <mesh filename="package://susan_description/meshes/mg6012-i36v3-5.stl"/>
@@ -873,5 +873,5 @@
 </visual>
 <collision>
-<origin xyz="1.3267518160498689285e-15 -0.0022999999999988637173 -0.047000000000000048683" rpy="1.570796326794896558 2.2208773040168372319e-16 1.5707963267948341635" />
+<origin xyz="1.3263601752762148032e-15 -0.0022999999999988697888 -0.047000000000000034805" rpy="1.570796326794896558 2.2208773040168411762e-16 1.5707963267948341635" />
 <geometry>
 <mesh filename="package://susan_description/meshes/mg6012-i36v3-5.stl"/>
@@ -879,5 +879,5 @@
 </collision>
 <visual>
-<origin xyz="1.3267518160498689285e-15 -0.0022999999999988637173 -0.047000000000000048683" rpy="1.570796326794896558 2.2208773040168372319e-16 1.5707963267948341635" />
+<origin xyz="1.3263601752762148032e-15 -0.0022999999999988697888 -0.047000000000000034805" rpy="1.570796326794896558 2.2208773040168411762e-16 1.5707963267948341635" />
 <geometry>
 <mesh filename="package://susan_description/meshes/mg6012-i36v3-15.stl"/>
@@ -888,5 +888,5 @@
 </visual>
 <collision>
-<origin xyz="1.3267518160498689285e-15 -0.0022999999999988637173 -0.047000000000000048683" rpy="1.570796326794896558 2.2208773040168372319e-16 1.5707963267948341635" />
+<origin xyz="1.3263601752762148032e-15 -0.0022999999999988697888 -0.047000000000000034805" rpy="1.570796326794896558 2.2208773040168411762e-16 1.5707963267948341635" />
 <geometry>
 <mesh filename="package://susan_description/meshes/mg6012-i36v3-15.stl"/>
@@ -894,5 +894,5 @@
 </collision>
 <visual>
-<origin xyz="1.3267518160498689285e-15 -0.0022999999999988637173 -0.047000000000000048683" rpy="1.570796326794896558 2.2208773040168372319e-16 1.5707963267948341635" />
+<origin xyz="1.3263601752762148032e-15 -0.0022999999999988697888 -0.047000000000000034805" rpy="1.570796326794896558 2.2208773040168411762e-16 1.5707963267948341635" />
 <geometry>
 <mesh filename="package://susan_description/meshes/mg6012-i36v3-23.stl"/>
@@ -903,5 +903,5 @@
 </visual>
 <collision>
-<origin xyz="1.3267518160498689285e-15 -0.0022999999999988637173 -0.047000000000000048683" rpy="1.570796326794896558 2.2208773040168372319e-16 1.5707963267948341635" />
+<origin xyz="1.3263601752762148032e-15 -0.0022999999999988697888 -0.047000000000000034805" rpy="1.570796326794896558 2.2208773040168411762e-16 1.5707963267948341635" />
 <geometry>
 <mesh filename="package://susan_description/meshes/mg6012-i36v3-23.stl"/>
@@ -909,5 +909,5 @@
 </collision>
 <visual>
-<origin xyz="1.3267518160498689285e-15 -0.0022999999999988637173 -0.047000000000000048683" rpy="1.570796326794896558 2.2208773040168372319e-16 1.5707963267948341635" />
+<origin xyz="1.3263601752762148032e-15 -0.0022999999999988697888 -0.047000000000000034805" rpy="1.570796326794896558 2.2208773040168411762e-16 1.5707963267948341635" />
 <geometry>
 <mesh filename="package://susan_description/meshes/mg6012-i36v3-14.stl"/>
@@ -918,5 +918,5 @@
 </visual>
 <collision>
-<origin xyz="1.3267518160498689285e-15 -0.0022999999999988637173 -0.047000000000000048683" rpy="1.570796326794896558 2.2208773040168372319e-16 1.5707963267948341635" />
+<origin xyz="1.3263601752762148032e-15 -0.0022999999999988697888 -0.047000000000000034805" rpy="1.570796326794896558 2.2208773040168411762e-16 1.5707963267948341635" />
 <geometry>
 <mesh filename="package://susan_description/meshes/mg6012-i36v3-14.stl"/>
@@ -924,5 +924,5 @@
 </collision>
 <visual>
-<origin xyz="1.3267518160498689285e-15 -0.0022999999999988637173 -0.047000000000000048683" rpy="1.570796326794896558 2.2208773040168372319e-16 1.5707963267948341635" />
+<origin xyz="1.3263601752762148032e-15 -0.0022999999999988697888 -0.047000000000000034805" rpy="1.570796326794896558 2.2208773040168411762e-16 1.5707963267948341635" />
 <geometry>
 <mesh filename="package://susan_description/meshes/mg6012-i36v3-1.stl"/>
@@ -933,5 +933,5 @@
 </visual>
 <collision>
-<origin xyz="1.3267518160498689285e-15 -0.0022999999999988637173 -0.047000000000000048683" rpy="1.570796326794896558 2.2208773040168372319e-16 1.5707963267948341635" />
+<origin xyz="1.3263601752762148032e-15 -0.0022999999999988697888 -0.047000000000000034805" rpy="1.570796326794896558 2.2208773040168411762e-16 1.5707963267948341635" />
 <geometry>
 <mesh filename="package://susan_description/meshes/mg6012-i36v3-1.stl"/>
@@ -939,5 +939,5 @@
 </collision>
 <visual>
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